File: Electrical/NMEA-2000-influxdb.kicad_sch (KiCad schematic)
At the start: 13 parts, among them J1 Conn_01x04, J2 Conn_01x04, J3 Conn_02x04, U1 LM7805_TO220, U2 ESP32_NODEMCU, U3 RTC-Module, U4 SD-Card-Module, U5 SN65HVD230

Commit message: Updated Schematic
Parts:
- U1: footprint Heatsinks:Heatsink_TO220-3_30x25x25mm -> Package_TO_SOT_THT:TO-220-3_Vertical
Connections:
- net +5V: now also U3.2 (VCC); no longer U3.1 (VCC)
- net GND: now also U3.1 (GND); no longer U3.2 (GND)
- net SCL: now also U3.3 (SDA); no longer U3.4 (SCL)
- net SDA: now also U3.4 (SCL); no longer U3.3 (SDA)
Changed lines of the file:
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@@
 	)
 	(no_connect
-		(at 262.89 80.01)
-	)
-	(no_connect
 		(at 99.06 52.07)
 	)
@@
 	)
 	(no_connect
-		(at 99.06 80.01)
+		(at 262.89 69.85)
 	)
 	(no_connect
-		(at 262.89 77.47)
+		(at 262.89 67.31)
+	)
+	(no_connect
+		(at 99.06 80.01)
 	)
 	(no_connect
@@
 	(wire
 		(pts
-			(xy 262.89 80.01) (xy 257.81 80.01)
+			(xy 147.32 62.23) (xy 154.94 62.23)
 		)
 		(stroke
@@
 	(wire
 		(pts
-			(xy 147.32 62.23) (xy 154.94 62.23)
+			(xy 262.89 67.31) (xy 257.81 67.31)
 		)
 		(stroke
@@
 	(wire
 		(pts
-			(xy 147.32 59.69) (xy 154.94 59.69)
+			(xy 257.81 77.47) (xy 265.43 77.47)
 		)
 		(stroke
@@
 	(wire
 		(pts
-			(xy 265.43 101.6) (xy 265.43 114.3)
+			(xy 147.32 59.69) (xy 154.94 59.69)
 		)
 		(stroke
@@
 	(wire
 		(pts
-			(xy 99.06 67.31) (xy 106.68 67.31)
+			(xy 265.43 101.6) (xy 265.43 114.3)
 		)
 		(stroke
@@
 	(wire
 		(pts
-			(xy 265.43 69.85) (xy 265.43 82.55)
+			(xy 99.06 67.31) (xy 106.68 67.31)
 		)
 		(stroke
@@
 	(wire
 		(pts
+			(xy 265.43 80.01) (xy 257.81 80.01)
+		)
+		(stroke
+			(width 0)
+			(type default)
+		)
+	)
+	(wire
+		(pts
 			(xy 82.55 36.83) (xy 82.55 39.37)
 		)
@@
 	(wire
 		(pts
-			(xy 262.89 77.47) (xy 257.81 77.47)
-		)
-		(stroke
-			(width 0)
-			(type default)
-		)
-	)
-	(wire
-		(pts
 			(xy 151.13 107.95) (xy 151.13 110.49)
 		)
@@
 	(wire
 		(pts
-			(xy 265.43 66.04) (xy 265.43 67.31)
+			(xy 123.19 135.89) (xy 123.19 140.97)
 		)
 		(stroke
@@
 	(wire
 		(pts
-			(xy 123.19 135.89) (xy 123.19 140.97)
+			(xy 99.06 92.71) (xy 106.68 92.71)
 		)
 		(stroke
@@
 	(wire
 		(pts
-			(xy 99.06 92.71) (xy 106.68 92.71)
+			(xy 72.39 36.83) (xy 72.39 39.37)
 		)
 		(stroke
@@
 	(wire
 		(pts
-			(xy 72.39 36.83) (xy 72.39 39.37)
+			(xy 120.65 153.67) (xy 128.27 153.67)
 		)
 		(stroke
@@
 	(wire
 		(pts
-			(xy 120.65 153.67) (xy 128.27 153.67)
+			(xy 140.97 156.21) (xy 148.59 156.21)
 		)
 		(stroke
@@
 	(wire
 		(pts
-			(xy 140.97 156.21) (xy 148.59 156.21)
+			(xy 120.65 143.51) (xy 128.27 143.51)
 		)
 		(stroke
@@
 	(wire
 		(pts
-			(xy 120.65 143.51) (xy 128.27 143.51)
+			(xy 147.32 80.01) (xy 154.94 80.01)
 		)
 		(stroke
@@
 	(wire
 		(pts
-			(xy 147.32 80.01) (xy 154.94 80.01)
+			(xy 265.43 82.55) (xy 265.43 80.01)
 		)
 		(stroke
@@
 	(wire
 		(pts
-			(xy 27.94 35.56) (xy 27.94 38.1)
+			(xy 262.89 69.85) (xy 257.81 69.85)
 		)
 		(stroke
@@
 	(wire
 		(pts
-			(xy 30.48 67.31) (xy 25.4 67.31)
+			(xy 27.94 35.56) (xy 27.94 38.1)
 		)
 		(stroke
@@
 	(wire
 		(pts
-			(xy 72.39 26.67) (xy 72.39 29.21)
+			(xy 30.48 67.31) (xy 25.4 67.31)
 		)
 		(stroke
@@
 	(wire
 		(pts
-			(xy 257.81 67.31) (xy 265.43 67.31)
+			(xy 72.39 26.67) (xy 72.39 29.21)
 		)
 		(stroke
@@
 	(wire
 		(pts
-			(xy 148.59 156.21) (xy 148.59 158.75)
+			(xy 265.43 63.5) (xy 265.43 77.47)
 		)
 		(stroke
@@
 	(wire
 		(pts
-			(xy 257.81 69.85) (xy 265.43 69.85)
+			(xy 148.59 156.21) (xy 148.59 158.75)
 		)
 		(stroke
@@
 	)
 	(symbol
-		(lib_id "power:+12V")
-		(at 72.39 26.67 0)
+		(lib_id "power:+5V")
+		(at 265.43 63.5 0)
 		(unit 1)
 		(exclude_from_sim no)
@@
 		(dnp no)
 		(fields_autoplaced yes)
-		(property "Reference" "#PWR02"
-			(at 72.39 30.48 0)
+		(property "Reference" "#PWR09"
+			(at 265.43 67.31 0)
 			(effects
 				(font
@@
 			)
 		)
-		(property "Value" "+12V"
-			(at 72.39 22.225 0)
+		(property "Value" "+5V"
+			(at 267.97 62.23 0)
 			(effects
 				(font
 					(size 1.27 1.27)
 				)
+				(justify left)
 			)
 		)
 		(property "Footprint" ""
-			(at 72.39 26.67 0)
+			(at 265.43 63.5 0)
 			(effects
 				(font
@@
 		)
 		(property "Datasheet" ""
-			(at 72.39 26.67 0)
+			(at 265.43 63.5 0)
 			(effects
 				(font
@@
 		)
 		(property "Description" ""
-			(at 72.39 26.67 0)
+			(at 265.43 63.5 0)
 			(effects
 				(font
@@
 			(project "NMEA-2000-influxdb"
 				(path "/efe7a42c-525a-4afc-8476-4cc785240ca6"
-					(reference "#PWR02")
+					(reference "#PWR09")
 					(unit 1)
 				)
@@
 	)
 	(symbol
-		(lib_id "power:+5V")
-		(at 265.43 66.04 0)
+		(lib_id "power:+12V")
+		(at 72.39 26.67 0)
 		(unit 1)
 		(exclude_from_sim no)
@@
 		(dnp no)
 		(fields_autoplaced yes)
-		(property "Reference" "#PWR09"
-			(at 265.43 69.85 0)
+		(property "Reference" "#PWR02"
+			(at 72.39 30.48 0)
 			(effects
 				(font
@@
 			)
 		)
-		(property "Value" "+5V"
-			(at 267.97 64.77 0)
+		(property "Value" "+12V"
+			(at 72.39 22.225 0)
 			(effects
 				(font
 					(size 1.27 1.27)
 				)
-				(justify left)
 			)
 		)
 		(property "Footprint" ""
-			(at 265.43 66.04 0)
+			(at 72.39 26.67 0)
 			(effects
 				(font
@@
 		)
 		(property "Datasheet" ""
-			(at 265.43 66.04 0)
+			(at 72.39 26.67 0)
 			(effects
 				(font
@@
 		)
 		(property "Description" ""
-			(at 265.43 66.04 0)
+			(at 72.39 26.67 0)
 			(effects
 				(font
@@
 			(project "NMEA-2000-influxdb"
 				(path "/efe7a42c-525a-4afc-8476-4cc785240ca6"
-					(reference "#PWR09")
+					(reference "#PWR02")
 					(unit 1)
 				)
@@
 			)
 		)
-		(property "Footprint" "Heatsinks:Heatsink_TO220-3_30x25x25mm"
+		(property "Footprint" "Package_TO_SOT_THT:TO-220-3_Vertical"
 			(at 82.55 23.495 0)
 			(effects
