File: Electrical/NMEA-2000-influxdb.kicad_pcb (KiCad board)
At the start: 4 copper layers, 134.6 x 182.9 mm, 32 parts, among them J1 Conn_01x04, J2 Conn_01x04, J3 Conn_02x04_Top_Bottom, J4 Conn_02x04_Top_Bottom, U1 SD-Card-Module, U11 JM-S05422A-001, U2 LM7805_TO220, U3 ESP32_NODEMCU, U4 SN65HVD230, U5 RTC-Module, U8 DA56-11CGKWA, U9 DA56-11CGKWA

Commit message: Added Mainboard
Parts:
- added D3: LED, LED_THT:LED_D5.0mm, F.Cu at (223.7, 183.8)
- added D4: LED, LED_THT:LED_D5.0mm, F.Cu at (236.5, 184.9)
- added D5: TJ-L5FYTXHTCYLCRGB-A5, LED_THT:LED_D5.0mm-4_RGB_Wide_Pins, F.Cu at (182.3, 202.7)
- added J5: Conn_01x04, TerminalBlock_Phoenix:TerminalBlock_Phoenix_MKDS-1,5-4-5.08_1x04_P5.08mm_Horizontal, F.Cu at (243.6, 204.7)
- added JP1: Jumper_2_Bridged, Connector_PinHeader_2.54mm:PinHeader_1x02_P2.54mm_Vertical, F.Cu at (172.5, 175.1)
- added JP10: Jumper_2_Open, Connector_PinHeader_2.54mm:PinHeader_1x02_P2.54mm_Vertical, F.Cu at (184.2, 76.2)
- added JP11: Jumper_3_Bridged12, Connector_PinHeader_2.54mm:PinHeader_1x03_P2.54mm_Vertical, F.Cu at (203.2, 74.9)
- added JP2: Jumper_2_Open, Connector_PinHeader_2.54mm:PinHeader_1x02_P2.54mm_Vertical, F.Cu at (177.1, 175.1)
- added JP3: Jumper_2_Bridged, Connector_PinHeader_2.54mm:PinHeader_1x02_P2.54mm_Vertical, F.Cu at (181.8, 175.1)
- added JP4: Jumper_2_Bridged, Connector_PinHeader_2.54mm:PinHeader_1x02_P2.54mm_Vertical, F.Cu at (186.4, 175.1)
- added JP5: Jumper_2_Bridged, Connector_PinHeader_2.54mm:PinHeader_1x02_P2.54mm_Vertical, F.Cu at (191.1, 175.1)
- added JP6: Jumper_2_Bridged, Connector_PinHeader_2.54mm:PinHeader_1x02_P2.54mm_Vertical, F.Cu at (195.7, 175.1)
- added JP7: Jumper_2_Bridged, Connector_PinHeader_2.54mm:PinHeader_1x02_P2.54mm_Vertical, F.Cu at (200.4, 175.1)
- added JP8: Jumper_2_Open, Connector_PinHeader_2.54mm:PinHeader_1x02_P2.54mm_Vertical, F.Cu at (205.0, 175.1)
- added JP9: Jumper_2_Bridged, Connector_PinHeader_2.54mm:PinHeader_1x02_P2.54mm_Vertical, F.Cu at (209.7, 175.1)
- added R14: 22R, Resistor_THT:R_Axial_DIN0204_L3.6mm_D1.6mm_P5.08mm_Horizontal, F.Cu at (187.7, 184.7)
- added R15: 38k, Resistor_THT:R_Axial_DIN0204_L3.6mm_D1.6mm_P5.08mm_Horizontal, F.Cu at (187.7, 187.9)
- added R16: 47k, Resistor_THT:R_Axial_DIN0204_L3.6mm_D1.6mm_P5.08mm_Horizontal, F.Cu at (187.7, 191.0)
- added R17: 38k, Resistor_THT:R_Axial_DIN0204_L3.6mm_D1.6mm_P5.08mm_Horizontal, F.Cu at (187.7, 194.2)
- added R18: 47k, Resistor_THT:R_Axial_DIN0204_L3.6mm_D1.6mm_P5.08mm_Horizontal, F.Cu at (187.7, 197.3)
- added R19: 120R, Resistor_THT:R_Axial_DIN0204_L3.6mm_D1.6mm_P5.08mm_Horizontal, F.Cu at (196.8, 76.2)
- added SW1: SW_Push, Button_Switch_THT:SW_PUSH_6mm_H13mm, F.Cu at (172.2, 200.9)
- added SW2: SW_Push, Button_Switch_THT:SW_PUSH_6mm_H13mm, F.Cu at (172.2, 209.5)
- D2: value LED_ABGR -> LED; footprint LED_THT:LED_D5.0mm-4_RGB_Wide_Pins -> LED_THT:LED_D5.0mm
- J3: value Conn_02x04_Top_Bottom -> Conn_02x04
- J4: value Conn_02x04_Top_Bottom -> Conn_02x04; moved to F.Cu
- R1, R2, R3, R4: value 38k -> 220R; moved to F.Cu
- R10: value 22R -> R; moved to F.Cu
- R11, U10, U7: moved to F.Cu
- R12: value R -> 38k; moved to F.Cu
- R13: value R -> 47k; moved to F.Cu
- R5: value 47k -> R; moved to F.Cu
- R6, R7: value 47k -> 38k; moved to F.Cu
- R8: value 22R -> 38k; moved to F.Cu
- R9: value R -> 22R; moved to F.Cu
- U1: value SD-Card-Module -> LM7805_TO220; footprint Connector_PinSocket_2.54mm:PinSocket_1x06_P2.54mm_Horizontal -> Package_TO_SOT_THT:TO-220-3_Vertical
- U11: value JM-S05422A-001 -> ~; footprint Display_7Segment:DA56-11CGKWA -> Package_SO:SSOP-28_3.9x9.9mm_P0.635mm
- U2: value LM7805_TO220 -> ESP32_NODEMCU; footprint Heatsinks:Heatsink_TO220-3_30x25x25mm -> esp32:esp32
- U3: value ESP32_NODEMCU -> RTC-Module; footprint esp32:esp32 -> Connector_PinSocket_2.54mm:PinSocket_1x06_P2.54mm_Horizontal
- U4: value SN65HVD230 -> SD-Card-Module; footprint Package_SO:SOIC-8_3.9x4.9mm_P1.27mm -> Connector_PinSocket_2.54mm:PinSocket_1x06_P2.54mm_Horizontal
- U5: value RTC-Module -> SN65HVD230; footprint Connector_PinSocket_2.54mm:PinSocket_1x06_P2.54mm_Horizontal -> Package_SO:SOIC-8_3.9x4.9mm_P1.27mm
- U6: value ~ -> DA56-11CGKWA; footprint Package_SO:SSOP-28_3.9x9.9mm_P0.635mm -> Display_7Segment:DA56-11CGKWA; moved to F.Cu
- U8: value DA56-11CGKWA -> JM-S05422A-001
- moved R12 103.8 mm to (179.6, 197.3), turned to 0 degrees
- moved U4 90.2 mm to (262.4, 95.9), turned to 180 degrees
- moved U9 88.3 mm to (265.4, 224.8), turned to 0 degrees
- moved D1 66.9 mm to (208.7, 183.8)
- moved J4 65.8 mm to (198.4, 208.7)
- moved U11 63.1 mm to (226.1, 193.3), turned to 0 degrees
- moved R13 62.8 mm to (187.7, 181.6), turned to 0 degrees
- moved C2 56.5 mm to (186.1, 99.1), turned to 0 degrees
- moved C1 55.7 mm to (200.7, 89.5), turned to 0 degrees
- moved U8 53.9 mm to (244.7, 224.8), turned to 0 degrees
- moved U3 51.8 mm to (262.3, 74.9), turned to 180 degrees
- moved R1 48.8 mm to (171.6, 181.6), turned to 0 degrees
- moved U2 47.2 mm to (230.0, 82.5)
- moved R2 45.2 mm to (171.6, 184.7), turned to 0 degrees
- moved U10 43.2 mm to (218.1, 193.3), turned to 0 degrees
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Connections:
- D1 pad 1: /Display/WIFI -> /Display/CAN_ST
- D2 pad 1: Net-(D2-A) -> /Display/SD_ST
- D2 pad 2: /Display/BLUE -> Net-(D2-A)
- J1 pad 2: CAN_L -> /CAN_H
- J1 pad 3: CAN_H -> /CAN_L
- J3 pad 1: +3V3 -> +5V
- J3 pad 10: unconnected-(J3-Pin_10-Pad10) -> /SD_ST
- J3 pad 11: /WIFI -> /RTC_ST
- J3 pad 12: /RED -> /WIFI_ST
- J3 pad 13: /GREEN -> /RED
- J3 pad 14: /BLUE -> /GREEN
- J3 pad 15: unconnected-(J3-Pin_15-Pad15) -> /BLUE
- J3 pad 16: unconnected-(J3-Pin_16-Pad16) -> GND
- J3 pad 2: unconnected-(J3-Pin_2-Pad2) -> +3V3
- J3 pad 3: unconnected-(J3-Pin_3-Pad3) -> /CAN_H
- J3 pad 4: SCL -> /CAN_L
- J3 pad 5: SDA -> /SCL
- J3 pad 6: unconnected-(J3-Pin_6-Pad6) -> /SDA
- J3 pad 7: unconnected-(J3-Pin_7-Pad7) -> /SW_TG
- J3 pad 8: GND -> /SW_CY
- J3 pad 9: unconnected-(J3-Pin_9-Pad9) -> /CAN_ST
- J4 pad 1: +3.3V -> +5VD
- J4 pad 10: unconnected-(J4-Pin_10-Pad10) -> /Display/SD_ST
- J4 pad 11: /Display/WIFI -> /Display/RTC_ST
- J4 pad 12: /Display/RED -> /Display/WIFI_ST
- J4 pad 13: /Display/GREEN -> /Display/RED
- J4 pad 14: /Display/BLUE -> /Display/GREEN
- J4 pad 15: unconnected-(J4-Pin_15-Pad15) -> /Display/BLUE
- J4 pad 16: unconnected-(J4-Pin_16-Pad16) -> GND1
- J4 pad 2: unconnected-(J4-Pin_2-Pad2) -> +3.3V
- J4 pad 3: unconnected-(J4-Pin_3-Pad3) -> /Display/CAN_H
- J4 pad 4: /Display/SCL -> /Display/CAN_L
- J4 pad 5: /Display/SDA -> /Display/SCL
- J4 pad 6: unconnected-(J4-Pin_6-Pad6) -> /Display/SDA
- J4 pad 7: unconnected-(J4-Pin_7-Pad7) -> /Display/SW_TG
- J4 pad 8: GND1 -> /Display/SW_CY
- J4 pad 9: unconnected-(J4-Pin_9-Pad9) -> /Display/CAN_ST
- R1 pad 1: unconnected-(R1-Pad1) -> +3.3V
- R1 pad 2: Net-(U6-ROW0/A2) -> Net-(D1-A)
- R10 pad 1: Net-(U10-COM2/KS1) -> Net-(U11-COM1/KS0)
- R10 pad 2: Net-(U11-COM2) -> Net-(U8-COM1)
- R11 pad 1: Net-(U10-COM2/KS1) -> Net-(U11-COM2/KS1)
- R11 pad 2: Net-(U11-COM2) -> Net-(U8-COM2)
- R12 pad 1: +3.3V -> Net-(U10-COM0/AD)
- R12 pad 2: Net-(D1-A) -> Net-(JP4-A)
- R13 pad 1: +3.3V -> Net-(U11-COM0/AD)
- R13 pad 2: Net-(D2-A) -> Net-(JP5-A)
- R2 pad 1: unconnected-(R1-Pad1) -> +3.3V
- R2 pad 2: Net-(U6-ROW2/A0) -> Net-(D2-A)
- R3 pad 1: unconnected-(R3-Pad1) -> +3.3V
- R3 pad 2: Net-(U7-ROW0/A2) -> Net-(D3-A)
- R4 pad 1: unconnected-(R3-Pad1) -> +3.3V
- R4 pad 2: Net-(U7-ROW1/A1) -> Net-(D4-A)
- R5 pad 1: Net-(U10-COM0/AD) -> +3.3V
- R5 pad 2: Net-(U10-ROW2/A0) -> Net-(D5-A)
- R6 pad 1: Net-(U10-COM0/AD) -> Net-(U7-COM0/AD)
- R6 pad 2: Net-(U10-ROW1/A1) -> Net-(JP1-A)
- R7 pad 1: Net-(U10-COM0/AD) -> Net-(U7-COM0/AD)
- R7 pad 2: Net-(U10-ROW0/A2) -> Net-(JP2-A)
- R8 pad 1: Net-(U10-COM1/KS0) -> Net-(U7-COM0/AD)
- R8 pad 2: Net-(U11-COM1) -> Net-(JP3-A)
- R9 pad 1: Net-(U10-COM1/KS0) -> Net-(U11-COM1/KS0)
- R9 pad 2: Net-(U11-COM1) -> Net-(U8-COM1)
- U1 pad 1: GND -> +12V
- U1 pad 2: +5V -> GND
- U1 pad 3: /MISO -> +5V
- U10 pad 10: unconnected-(U10-ROW15/K13/INT-Pad10) -> Net-(U10-ROW15/K13/INT)
- U10 pad 23: Net-(U10-ROW2/A0) -> Net-(JP8-B)
- U10 pad 24: Net-(U10-ROW1/A1) -> Net-(JP6-B)
- U10 pad 25: Net-(U10-ROW0/A2) -> Net-(JP4-B)
- U11 pad 1: Net-(U10-ROW0/A2) -> GND1
- U11 pad 10: Net-(U10-ROW8/K6) -> unconnected-(U11-ROW15/K13/INT-Pad10)
- U11 pad 11: Net-(U11-COM1) -> Net-(U11-ROW14/K12)
- U11 pad 12: Net-(U10-ROW10/K8) -> Net-(U11-ROW13/K11)
- U11 pad 13: Net-(U10-ROW9/K7) -> Net-(U11-ROW12/K10)
- U11 pad 14: Net-(U10-ROW11/K9) -> Net-(U11-ROW11/K9)
- U11 pad 15: Net-(U10-ROW12/K10) -> Net-(U11-ROW10/K8)
- U11 pad 16: Net-(U11-COM2) -> Net-(U11-ROW9/K7)
- U11 pad 17: Net-(U10-ROW13/K11) -> Net-(U11-ROW8/K6)
- U11 pad 18: Net-(U10-ROW14/K12) -> Net-(U11-ROW7/K5)
- U11 pad 2: Net-(U10-ROW1/A1) -> Net-(U11-COM0/AD)
- U11 pad 3: unconnected-(U11-NC-Pad3) -> Net-(U11-COM1/KS0)
- U11 pad 4: Net-(U10-ROW2/A0) -> Net-(U11-COM2/KS1)
- U11 pad 5: Net-(U10-ROW3/K1) -> unconnected-(U11-COM3/KS2-Pad5)
- U11 pad 6: Net-(U10-ROW4/K2) -> unconnected-(U11-COM4-Pad6)
- U11 pad 7: Net-(U10-ROW5/K3) -> unconnected-(U11-COM5-Pad7)
- U11 pad 8: Net-(U10-ROW6/K4) -> unconnected-(U11-COM6-Pad8)
- U11 pad 9: Net-(U10-ROW7/K5) -> unconnected-(U11-COM7-Pad9)
- U2 pad 1: +12V -> +5V
- U2 pad 2: GND -> unconnected-(U2-CMD-Pad2)
- U2 pad 3: +5V -> /MISO
- U3 pad 1: +5V -> GND
- U3 pad 2: unconnected-(U3-CMD-Pad2) -> +5V
- U3 pad 3: /MISO -> /SCL
- U3 pad 4: /MOSI -> /SDA
- U3 pad 6: GND -> unconnected-(U3-32K-Pad6)
- U4 pad 1: /CAN_RX -> GND
- U4 pad 2: GND -> +5V
- U4 pad 3: +3V3 -> /MISO
- U4 pad 4: /CAN_TX -> /MOSI
- U4 pad 5: unconnected-(U4-Vref-Pad5) -> /SCK
- U4 pad 6: CAN_L -> /CS
- U5 pad 1: +5V -> /CAN_RX
- U5 pad 3: SDA -> +3V3
- U5 pad 4: SCL -> /CAN_TX
- U5 pad 6: unconnected-(U5-32K-Pad6) -> /CAN_H
- U6 pad 1: GND1 -> Net-(U6-DIG1_E)
- U6 pad 10: Net-(U6-ROW15/K13/INT) -> Net-(U6-DIG2_B)
- U6 pad 11: Net-(U6-ROW14/K12) -> Net-(U6-DIG2_A)
- U6 pad 12: Net-(U6-ROW13/K11) -> Net-(JP3-B)
- U6 pad 13: Net-(U6-ROW12/K10) -> Net-(U6-DIG2_CA)
- U6 pad 14: Net-(U6-ROW11/K9) -> Net-(U6-DIG1_CA)
- U6 pad 15: Net-(U6-ROW10/K8) -> Net-(U6-DIG1_B)
- U6 pad 16: Net-(U6-ROW9/K7) -> Net-(U6-DIG1_A)
- U6 pad 17: Net-(U6-ROW8/K6) -> Net-(U6-DIG1_G)
- U6 pad 18: Net-(U6-ROW7/K5) -> Net-(U6-DIG1_F)
- U6 pad 2: unconnected-(R1-Pad1) -> Net-(U6-DIG1_D)
- U6 pad 3: Net-(U6-COM1/KS0) -> Net-(U6-DIG1_C)
- U6 pad 4: Net-(U6-COM2/KS1) -> Net-(U6-DP1)
- U6 pad 5: unconnected-(U6-COM3/KS2-Pad5) -> Net-(U6-DIG2_E)
- U6 pad 6: unconnected-(U6-COM4-Pad6) -> Net-(U6-DIG2_D)
- U6 pad 7: unconnected-(U6-COM5-Pad7) -> Net-(JP2-B)
- U6 pad 8: unconnected-(U6-COM6-Pad8) -> Net-(U6-DIG2_C)
- U6 pad 9: unconnected-(U6-COM7-Pad9) -> Net-(JP1-B)
- U7 pad 10: Net-(U7-ROW15/K13/INT) -> Net-(U6-DP1)
- U7 pad 11: Net-(U7-ROW14/K12) -> Net-(U6-DIG1_G)
- U7 pad 12: Net-(U7-ROW13/K11) -> Net-(U6-DIG1_F)
- U7 pad 13: Net-(U7-ROW12/K10) -> Net-(U6-DIG1_E)
- U7 pad 14: Net-(U7-ROW11/K9) -> Net-(U6-DIG1_D)
- U7 pad 15: Net-(U7-ROW10/K8) -> Net-(U6-DIG1_C)
- U7 pad 16: Net-(U7-ROW9/K7) -> Net-(U6-DIG1_B)
- U7 pad 17: Net-(U7-ROW8/K6) -> Net-(U6-DIG1_A)
- U7 pad 18: Net-(U7-ROW7/K5) -> Net-(U6-DIG2_A)
- U7 pad 19: Net-(U7-ROW6/K4) -> Net-(U6-DIG2_B)
- U7 pad 2: unconnected-(R3-Pad1) -> Net-(U7-COM0/AD)
- U7 pad 20: Net-(U7-ROW5/K3) -> Net-(U6-DIG2_C)
- U7 pad 21: Net-(U7-ROW4/K2) -> Net-(U6-DIG2_D)
- U7 pad 22: Net-(U7-ROW3/K1) -> Net-(U6-DIG2_E)
- U7 pad 23: unconnected-(U7-ROW2/A0-Pad23) -> Net-(JP3-B)
- U7 pad 24: Net-(U7-ROW1/A1) -> Net-(JP2-B)
- U7 pad 25: Net-(U7-ROW0/A2) -> Net-(JP1-B)
- U7 pad 3: Net-(U7-COM1/KS0) -> Net-(U6-DIG2_CA)
- U7 pad 4: Net-(U7-COM2/KS1) -> Net-(U6-DIG1_CA)
- U8 pad 1: Net-(U6-ROW12/K10) -> Net-(JP9-B)
- U8 pad 10: Net-(U6-ROW6/K4) -> Net-(U11-ROW8/K6)
- U8 pad 11: Net-(U6-ROW7/K5) -> Net-(U8-COM1)
- U8 pad 12: Net-(U6-ROW2/A0) -> Net-(U11-ROW10/K8)
- U8 pad 13: Net-(U6-COM1/KS0) -> Net-(U11-ROW9/K7)
- U8 pad 14: Net-(U6-COM2/KS1) -> Net-(U11-ROW11/K9)
- U8 pad 15: Net-(U6-ROW9/K7) -> Net-(U11-ROW12/K10)
- U8 pad 16: Net-(U6-ROW8/K6) -> Net-(U8-COM2)
- U8 pad 17: Net-(U6-ROW14/K12) -> Net-(U11-ROW13/K11)
- U8 pad 18: Net-(U6-ROW13/K11) -> Net-(U11-ROW14/K12)
- U8 pad 2: Net-(U6-ROW11/K9) -> Net-(JP7-B)
- U8 pad 3: Net-(U6-ROW10/K8) -> unconnected-(U8-NC-Pad3)
- U8 pad 4: Net-(U6-ROW15/K13/INT) -> Net-(JP5-B)
- U8 pad 5: Net-(U6-ROW3/K1) -> Net-(U11-ROW3/K1)
- U8 pad 6: Net-(U6-ROW4/K2) -> Net-(U11-ROW4/K2)
- U8 pad 7: unconnected-(U6-ROW1/A1-Pad24) -> Net-(U11-ROW5/K3)
- U8 pad 8: Net-(U6-ROW5/K3) -> Net-(U11-ROW6/K4)
- U8 pad 9: Net-(U6-ROW0/A2) -> Net-(U11-ROW7/K5)
- U9 pad 1: Net-(U7-ROW12/K10) -> Net-(U10-ROW12/K10)
- U9 pad 10: Net-(U7-ROW6/K4) -> Net-(U10-ROW6/K4)
- U9 pad 11: Net-(U7-ROW7/K5) -> Net-(U10-ROW7/K5)
- U9 pad 12: unconnected-(U7-ROW2/A0-Pad23) -> Net-(JP8-B)
- U9 pad 13: Net-(U7-COM1/KS0) -> Net-(U10-COM1/KS0)
- U9 pad 14: Net-(U7-COM2/KS1) -> Net-(U10-COM2/KS1)
- U9 pad 15: Net-(U7-ROW9/K7) -> Net-(U10-ROW9/K7)
- U9 pad 16: Net-(U7-ROW8/K6) -> Net-(U10-ROW8/K6)
- U9 pad 17: Net-(U7-ROW14/K12) -> Net-(U10-ROW14/K12)
- U9 pad 18: Net-(U7-ROW13/K11) -> Net-(U10-ROW13/K11)
- U9 pad 2: Net-(U7-ROW11/K9) -> Net-(U10-ROW11/K9)
- U9 pad 3: Net-(U7-ROW10/K8) -> Net-(U10-ROW10/K8)
- U9 pad 4: Net-(U7-ROW15/K13/INT) -> Net-(U10-ROW15/K13/INT)
- U9 pad 5: Net-(U7-ROW3/K1) -> Net-(U10-ROW3/K1)
- U9 pad 6: Net-(U7-ROW4/K2) -> Net-(U10-ROW4/K2)
- U9 pad 7: Net-(U7-ROW1/A1) -> Net-(JP6-B)
- U9 pad 8: Net-(U7-ROW5/K3) -> Net-(U10-ROW5/K3)
- U9 pad 9: Net-(U7-ROW0/A2) -> Net-(JP4-B)
Routing:
- net GND: track 16.1 -> 267.5 mm, vias 1 -> 0
- net /Display/SDA: track 176.6 -> 0.00 mm, vias 2 -> 0
- net /CAN_L: track 0.00 -> 163.1 mm
- net /Display/SCL: track 159.4 -> 0.00 mm, vias 2 -> 0
- net /CAN_H: track 0.00 -> 121.6 mm
- net +5V: track 49.7 -> 152.0 mm, vias 1 -> 0
- net /RTC_ST: track 0.00 -> 91.3 mm
- net +3.3V: track 86.1 -> 0.00 mm, vias 1 -> 0
- net /SW_CY: track 0.00 -> 82.2 mm
- net /SCL: track 0.00 -> 81.3 mm
- net /SW_TG: track 0.00 -> 76.1 mm
- net /SD_ST: track 0.00 -> 74.3 mm
- net /CAN_ST: track 0.00 -> 73.4 mm
- net /SDA: track 0.00 -> 69.7 mm
- net SDA: track 61.5 -> 0.00 mm
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- removed copper zone on F.Cu, net +5VD
- removed copper zone on B.Cu, net GND1
Other:
- board size 134.6 x 182.9 mm -> 149.9 x 71.8 mm

Commit message: Added Mainboard
Parts:
- moved U3 3.78 mm to (262.3, 71.1)
Routing:
- net +5V: track 152.0 -> 129.1 mm
- net GND: track 267.5 -> 249.7 mm
- net /SCL: track 81.3 -> 70.2 mm
- net /CS: track 49.8 -> 58.2 mm
- net /SDA: track 69.7 -> 73.3 mm
Changed lines of the file:
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@@
 	(footprint "Connector_PinSocket_2.54mm:PinSocket_1x06_P2.54mm_Horizontal"
 		(layer "F.Cu")
-		(at 262.3 74.905 180)
+		(at 262.3 71.12 180)
 		(descr "Through hole angled socket strip, 1x06, 2.54mm pitch, 8.51mm socket length, single row (from Kicad 4.0.7), script generated")
 		(tags "Through hole angled socket strip THT 1x06 2.54mm single row")
@@
 	)
 	(segment
-		(start 256.54 73.025)
-		(end 259.055 75.54)
+		(start 208.22 89.535)
+		(end 208.22 79.95)
 		(width 0.25)
 		(layer "F.Cu")
@@
 	)
 	(segment
-		(start 256.54 67.31)
-		(end 256.54 73.025)
+		(start 180.676 93.98)
+		(end 175.133 88.437)
 		(width 0.25)
 		(layer "F.Cu")
@@
 	)
 	(segment
-		(start 180.676 93.98)
-		(end 175.133 88.437)
+		(start 208.22 79.95)
+		(end 203.2 74.93)
 		(width 0.25)
 		(layer "F.Cu")
@@
 	)
 	(segment
-		(start 248.92 59.69)
-		(end 256.54 67.31)
-		(width 0.25)
-		(layer "F.Cu")
-		(net 2)
-	)
-	(segment
 		(start 193.04 88.9)
 		(end 187.96 93.98)
@@
 	)
 	(segment
-		(start 259.055 75.54)
-		(end 262.3 75.54)
-		(width 0.25)
-		(layer "F.Cu")
-		(net 2)
-	)
-	(segment
 		(start 283.845 96.52)
 		(end 280.035 92.71)
@@
 	)
 	(segment
-		(start 262.3 75.54)
-		(end 267.335 80.575)
-		(width 0.25)
+		(start 262.3 71.12)
+		(end 258.445 71.12)
+		(width 0.3)
 		(layer "F.Cu")
 		(net 2)
@@
 	)
 	(segment
+		(start 258.445 71.12)
+		(end 256.54 73.025)
+		(width 0.3)
+		(layer "F.Cu")
+		(net 2)
+	)
+	(segment
 		(start 254.635 74.93)
 		(end 242.678 74.93)
@@
 	)
 	(segment
-		(start 267.335 80.575)
-		(end 267.335 92.71)
-		(width 0.25)
-		(layer "F.Cu")
-		(net 2)
-	)
-	(segment
 		(start 194.945 95.25)
 		(end 193.615 96.58)
@@
 	)
 	(segment
-		(start 242.678 59.69)
-		(end 248.92 59.69)
-		(width 0.25)
-		(layer "F.Cu")
-		(net 2)
-	)
-	(segment
 		(start 213.995 92.71)
 		(end 217.678 92.71)
@@
 	)
 	(segment
-		(start 203.2 74.93)
-		(end 203.2 84.515)
-		(width 0.25)
-		(layer "In1.Cu")
+		(start 250.87 59.69)
+		(end 242.678 59.69)
+		(width 0.3)
+		(layer "In2.Cu")
 		(net 2)
 	)
 	(segment
-		(start 203.2 84.515)
-		(end 208.22 89.535)
-		(width 0.25)
-		(layer "In1.Cu")
+		(start 262.3 71.12)
+		(end 250.87 59.69)
+		(width 0.3)
+		(layer "In2.Cu")
 		(net 2)
 	)
@@
 	)
 	(segment
-		(start 262.427 93.32)
-		(end 265.43 90.317)
-		(width 0.25)
-		(layer "B.Cu")
-		(net 3)
-	)
-	(segment
 		(start 186.115 99.06)
 		(end 186.115 93.285)
@@
 	)
 	(segment
-		(start 265.43 90.317)
-		(end 265.43 76.13)
-		(width 0.25)
-		(layer "B.Cu")
-		(net 3)
-	)
-	(segment
-		(start 265.43 76.13)
-		(end 262.3 73)
-		(width 0.25)
-		(layer "B.Cu")
-		(net 3)
-	)
-	(segment
 		(start 190.5 88.9)
 		(end 190.5 89.535)
@@
 	)
 	(segment
-		(start 254.147 91.44)
-		(end 221.488 91.44)
+		(start 262.427 83.16)
+		(end 243.987 101.6)
 		(width 0.25)
 		(layer "F.Cu")
@@
 	)
 	(segment
-		(start 262.427 83.16)
-		(end 254.147 91.44)
+		(start 243.987 101.6)
+		(end 231.648 101.6)
 		(width 0.25)
 		(layer "F.Cu")
@@
 	)
 	(segment
-		(start 221.488 91.44)
+		(start 231.648 101.6)
 		(end 217.678 87.63)
 		(width 0.25)
@@
 	)
 	(segment
-		(start 249.625 57.785)
-		(end 241.3 57.785)
-		(width 0.25)
-		(layer "F.Cu")
-		(net 22)
-	)
-	(segment
-		(start 241.3 64.77)
-		(end 242.678 64.77)
-		(width 0.25)
-		(layer "F.Cu")
-		(net 22)
-	)
-	(segment
-		(start 240.03 59.055)
-		(end 240.03 63.5)
-		(width 0.25)
-		(layer "F.Cu")
-		(net 22)
-	)
-	(segment
-		(start 240.03 63.5)
-		(end 241.3 64.77)
-		(width 0.25)
-		(layer "F.Cu")
+		(start 269.875 107.4325)
+		(end 269.875 67.31)
+		(width 0.3)
+		(layer "In2.Cu")
 		(net 22)
 	)
 	(segment
-		(start 241.3 57.785)
-		(end 240.03 59.055)
-		(width 0.25)
-		(layer "F.Cu")
+		(start 271.145 108.7025)
+		(end 269.875 107.4325)
+		(width 0.3)
+		(layer "In2.Cu")
 		(net 22)
 	)
 	(segment
-		(start 262.3 70.46)
-		(end 249.625 57.785)
-		(width 0.25)
-		(layer "F.Cu")
+		(start 268.605 66.04)
+		(end 262.3 66.04)
+		(width 0.3)
+		(layer "In2.Cu")
 		(net 22)
 	)
 	(segment
-		(start 269.875 71.755)
-		(end 268.58 70.46)
-		(width 0.25)
+		(start 269.875 67.31)
+		(end 268.605 66.04)
+		(width 0.3)
 		(layer "In2.Cu")
 		(net 22)
 	)
 	(segment
-		(start 269.875 107.4325)
-		(end 269.875 71.755)
-		(width 0.25)
-		(layer "In2.Cu")
+		(start 262.3 66.04)
+		(end 252.73 66.04)
+		(width 0.3)
+		(layer "B.Cu")
 		(net 22)
 	)
 	(segment
-		(start 271.145 108.7025)
-		(end 269.875 107.4325)
-		(width 0.25)
-		(layer "In2.Cu")
+		(start 252.73 66.04)
+		(end 251.46 64.77)
+		(width 0.3)
+		(layer "B.Cu")
 		(net 22)
 	)
 	(segment
-		(start 268.58 70.46)
-		(end 262.3 70.46)
-		(width 0.25)
-		(layer "In2.Cu")
+		(start 251.46 64.77)
+		(end 242.678 64.77)
+		(width 0.3)
+		(layer "B.Cu")
 		(net 22)
 	)
@@
 	)
 	(segment
-		(start 269.875 67.945)
-		(end 262.325 67.945)
-		(width 0.25)
-		(layer "In2.Cu")
+		(start 249.609 72.39)
+		(end 242.678 72.39)
+		(width 0.3)
+		(layer "F.Cu")
 		(net 28)
 	)
 	(segment
-		(start 271.145 106.1625)
-		(end 271.145 69.215)
-		(width 0.25)
-		(layer "In2.Cu")
+		(start 258.499 63.5)
+		(end 249.609 72.39)
+		(width 0.3)
+		(layer "F.Cu")
 		(net 28)
 	)
 	(segment
-		(start 271.145 69.215)
-		(end 269.875 67.945)
-		(width 0.25)
-		(layer "In2.Cu")
+		(start 262.3 63.5)
+		(end 258.499 63.5)
+		(width 0.3)
+		(layer "F.Cu")
 		(net 28)
 	)
 	(segment
-		(start 262.325 67.945)
-		(end 262.3 67.92)
-		(width 0.25)
+		(start 262.3 63.5)
+		(end 268.605 63.5)
+		(width 0.3)
 		(layer "In2.Cu")
 		(net 28)
 	)
 	(segment
-		(start 259.08 71.755)
-		(end 258.445 72.39)
-		(width 0.25)
-		(layer "B.Cu")
-		(net 28)
-	)
-	(segment
-		(start 259.08 68.58)
-		(end 259.08 71.755)
-		(width 0.25)
-		(layer "B.Cu")
-		(net 28)
-	)
-	(segment
-		(start 262.3 67.92)
-		(end 259.74 67.92)
-		(width 0.25)
-		(layer "B.Cu")
-		(net 28)
-	)
-	(segment
-		(start 258.445 72.39)
-		(end 242.678 72.39)
-		(width 0.25)
-		(layer "B.Cu")
+		(start 271.145 66.04)
+		(end 271.145 106.1625)
+		(width 0.3)
+		(layer "In2.Cu")
 		(net 28)
 	)
 	(segment
-		(start 259.74 67.92)
-		(end 259.08 68.58)
-		(width 0.25)
-		(layer "B.Cu")
+		(start 268.605 63.5)
+		(end 271.145 66.04)
+		(width 0.3)
+		(layer "In2.Cu")
 		(net 28)
 	)

Commit message: Updated Schematic
Parts:
- removed D5: TJ-L5FYTXHTCYLCRGB-A5, LED_THT:LED_D5.0mm-4_RGB_Wide_Pins
- removed the J4 at (198.4, 208.7)
- removed J5: Conn_01x04, TerminalBlock_Phoenix:TerminalBlock_Phoenix_MKDS-1,5-4-5.08_1x04_P5.08mm_Horizontal
- removed the JP1 at (172.5, 175.1)
- removed the JP2 at (177.1, 175.1)
- removed JP3, JP4, JP5, JP6, JP7, JP9: Jumper_2_Bridged, Connector_PinHeader_2.54mm:PinHeader_1x02_P2.54mm_Vertical
- removed JP8: Jumper_2_Open, Connector_PinHeader_2.54mm:PinHeader_1x02_P2.54mm_Vertical
- removed R10: R, Resistor_THT:R_Axial_DIN0204_L3.6mm_D1.6mm_P5.08mm_Horizontal
- removed R11, R14, R9: 22R, Resistor_THT:R_Axial_DIN0204_L3.6mm_D1.6mm_P5.08mm_Horizontal
- removed R12, R15, R17, R6, R7, R8: 38k, Resistor_THT:R_Axial_DIN0204_L3.6mm_D1.6mm_P5.08mm_Horizontal
- removed R13, R16, R18: 47k, Resistor_THT:R_Axial_DIN0204_L3.6mm_D1.6mm_P5.08mm_Horizontal
- removed the R5 at (171.6, 194.2)
- removed SW1, SW2: SW_Push, Button_Switch_THT:SW_PUSH_6mm_H13mm
- removed U10, U11, U7: ~, Package_SO:SSOP-28_3.9x9.9mm_P0.635mm
- removed the U3 at (262.3, 71.1)
- removed U6, U9: DA56-11CGKWA, Display_7Segment:DA56-11CGKWA
- removed U8: JM-S05422A-001, Display_7Segment:DA56-11CGKWA
- added A1: LM2596_Step_Down_Module, LM2596:LM2596_Step_Down_Module-21.3x43.6mm, F.Cu at (166.7, 62.2)
- added J3: Conn_01x02, Connector_PinSocket_2.54mm:PinSocket_1x02_P2.54mm_Vertical, F.Cu at (107.4, 64.2)
- added U5: SN65HVD230-Module, Connector_PinSocket_2.54mm:PinSocket_1x04_P2.54mm_Horizontal, F.Cu at (74.4, 68.5)
- D1, D2, D3, D4: footprint LED_THT:LED_D5.0mm -> LED_THT:LED_D3.0mm
- J4: renamed from J3; value Conn_02x04 -> Conn_02x08
- R1: value 220R -> 1.5k
- R2: value 220R -> 1.2k
- R3: value 220R -> 500R
- R4: value 220R -> 330R
- moved D4 169.8 mm to (78.1, 123.8)
- moved D3 159.3 mm to (78.1, 119.3)
- moved D2 154.5 mm to (78.1, 114.7)
- moved D1 150.0 mm to (78.1, 110.1)
- moved R1 109.8 mm to (88.2, 110.1), turned to 180 degrees
- moved R2 108.9 mm to (88.2, 114.7), turned to 180 degrees
- moved R3 108.0 mm to (88.2, 119.3), turned to 180 degrees
- moved R4 107.1 mm to (88.2, 123.8), turned to 180 degrees
- moved J1 100.1 mm to (75.9, 76.4)
- moved J2 99.6 mm to (81.6, 96.6)
- moved U3 99.1 mm to (163.6, 102.6)
- moved U1 99.1 mm to (96.7, 95.7)
- moved C1 99.1 mm to (101.9, 96.3)
- moved J4 99.1 mm to (167.2, 115.5)
- moved JP1 99.1 mm to (85.3, 83.0)
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- renumbered JP10 to JP1, JP11 to JP2, R19 to R5, U4 to U3, U5 to U4
Connections:
- D1 pad 1: /Display/CAN_ST -> GND
- D2 pad 1: /Display/SD_ST -> GND
- D3 pad 1: /Display/RTC_ST -> GND
- D4 pad 1: /Display/WIFI_ST -> GND
- J1 pad 1: +12V -> VMot
- R1 pad 1: +3.3V -> VMot
- R2 pad 1: +3.3V -> +12V
- R3 pad 1: +3.3V -> +5V
- U2 pad 12: unconnected-(U2-G33-Pad12) -> /CAN_RX_B
- U2 pad 13: unconnected-(U2-G32-Pad13) -> /CAN_TX_B
Routing:
- net +12V: track 42.0 -> 229.0 mm
- net VMot: track 0.00 -> 143.4 mm
- net GND: track 249.7 -> 159.6 mm
- net +3.3V: track 0.00 -> 61.0 mm
- net /CAN_TX_B: track 0.00 -> 53.0 mm
- net /CAN_RX_B: track 0.00 -> 53.0 mm
- net /TX: track 91.1 -> 120.4 mm
- net /SCL: track 70.2 -> 93.7 mm
- net /CAN_H: track 121.6 -> 144.1 mm
- net /RX: track 83.9 -> 105.4 mm
- net /SDA: track 73.3 -> 52.8 mm
- net /CAN_L: track 163.1 -> 150.7 mm
- net +5V: track 129.1 -> 136.8 mm, vias 0 -> 2
- net Net-(D4-A): track 0.00 -> 2.54 mm
- net Net-(D3-A): track 0.00 -> 2.54 mm
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